File: v2/sch/motor_back.sch (EAGLE design)
At the start: 12 parts, among them K1 DTSM-62K-S-V-T/R, K2 DTSM-62K-S-V-T/R

Commit message: routing almost finished
Parts:
- added C2, C3: 4.7uF, rcl:C-EUC0805
- added R1, R2, R3: 1k, rcl:R-EU_R0603
Connections:
- new net BUTTONS: JP1.1, R1.1, R3.1
- new net GND: C2.1, C3.1, JP2.2, K1.B0, K1.B1, K2.B0, K2.B1, LED1.GND, LED2.GND, LED3.GND, LED4.GND, LED5.GND, LED6.GND, LED7.GND, LED8.GND
- new net N$1: LED1.DO, LED2.DI
- new net N$13: K1.A0, K1.A1, R1.2
- new net N$14: K2.A0, K2.A1, R2.2
- new net N$15: R2.1, R3.2
- new net N$2: LED2.DO, LED3.DI
- new net N$3: LED3.DO, LED4.DI
- new net N$4: LED4.DO, LED5.DI
- new net N$5: LED5.DO, LED6.DI
- new net N$6: LED6.DO, LED7.DI
- new net N$7: LED7.DO, LED8.DI
- new net NEOPIXEL: JP1.2, LED1.DI
- new net VDD: C2.2, C3.2, JP2.1, LED1.VDD, LED2.VDD, LED3.VDD, LED4.VDD, LED5.VDD, LED6.VDD, LED7.VDD, LED8.VDD
Other:
- moved on the sheet: K1, K2
