File: v2/sch/motor_back.brd (EAGLE design)
At the start: 93 x 30.8 mm, 12 parts, among them K1 DTSM-62K-S-V-T/R, K2 DTSM-62K-S-V-T/R

Commit message: routing almost finished
Parts:
- added C2, C3: 4.7uF, rcl:C0805
- added R1, R2, R3: 1k, rcl:R0603
- moved K1 0.60 mm to (9.27, 6.27)
- moved K2 0.60 mm to (80.9, 6.29)
- moved LED1 0.37 mm to (8.47, 14.6)
- moved LED5 0.26 mm to (53.8, 14.6)
- moved LED4 0.14 mm to (34.5, 14.6)
- moved LED2 0.11 mm to (13.4, 20.0)
- moved LED3 0.11 mm to (18.1, 14.6)
- moved LED6 0.06 mm to (72.1, 14.6)
- moved LED7 0.06 mm to (76.8, 20.0)
Connections:
- new net BUTTONS: JP1.1, R1.1, R3.1
- new net N$1: LED1.1-DOUT, LED2.3-DIN
- new net N$13: K1.1, K1.4, R1.2
- new net N$14: K2.1, K2.4, R2.2
- new net N$15: R2.1, R3.2
- new net N$2: LED2.1-DOUT, LED3.3-DIN
- new net N$3: LED3.1-DOUT, LED4.3-DIN
- new net N$4: LED4.1-DOUT, LED5.3-DIN
- new net N$5: LED5.1-DOUT, LED6.3-DIN
- new net N$6: LED6.1-DOUT, LED7.3-DIN
- new net N$7: LED7.1-DOUT, LED8.3-DIN
- new net NEOPIXEL: JP1.2, LED1.3-DIN
- net GND: now also C2.1, C3.1, JP2.2, K1.2, K1.3, K2.2, K2.3
- net VDD: now also C2.2, C3.2, JP2.1
Routing:
- net GND: track 0.00 -> 193.8 mm, vias 0 -> 4
- net VDD: track 0.00 -> 135.0 mm, vias 0 -> 10
- net BUTTONS: track 0.00 -> 58.9 mm, vias 0 -> 2
- net NEOPIXEL: track 0.00 -> 28.5 mm
- net N$5: track 0.00 -> 17.4 mm
- net N$4: track 0.00 -> 16.9 mm
- net N$3: track 0.00 -> 14.0 mm
- net N$14: track 0.00 -> 11.5 mm
- net N$13: track 0.00 -> 10.9 mm
- net N$1: track 0.00 -> 10.2 mm
- net N$6: track 0.00 -> 9.89 mm
- net N$2: track 0.00 -> 4.49 mm
- net N$7: track 0.00 -> 4.40 mm
- net N$15: track 0.00 -> 1.50 mm
- added copper zone on layer 1, net GND
- added copper zone on layer 16, net GND

Commit message: mid-update, fixing issues
Parts:
- moved C3 1.37 mm to (78.2, 24.2)
- moved JP2 1.37 mm to (73.2, 1.91)
- moved LED6 1.37 mm to (73.5, 14.6)
- moved LED7 1.37 mm to (78.2, 20.0)
- moved LED8 1.37 mm to (83.1, 14.6)
- moved R3 1.37 mm to (71.4, 9.00)
- moved JP1 1.37 mm to (19.9, 1.80)
- moved C2 1.37 mm to (14.8, 24.2)
- moved K1 1.37 mm to (10.6, 6.27)
- moved LED1 1.37 mm to (9.84, 14.6)
- moved LED2 1.37 mm to (14.8, 20.0)
- moved LED3 1.37 mm to (19.5, 14.6)
- moved LED4 1.37 mm to (35.9, 14.6)
- moved LED5 1.37 mm to (55.2, 14.6)
- moved R1 1.37 mm to (18.2, 9.00)
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Other:
- outline, holes or cut-outs redrawn
