File: v2/sch/bot_base.sch (EAGLE design)
At the start: 39 parts, among them K2 DTSM-62K-S-V-T/R, Q0 QWIIC_RIGHT_ANGLE, U1 ESP32-C3-MINI-1-N4, U4 LGS4084HB5

Commit message: update for most recent prototypes
Parts:
- added R14: 1K, rcl:R-EU_R0603
Connections:
- net GND: now also R14.1
- net MOTOR2A_LV: now also R14.2
Other:
- note added: "stops motor run in bootloader"
Changed lines of the file:
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@@
 <setting verticaltext="up"/>
 </settings>
-<grid distance="0.05" unitdist="inch" unit="inch" style="lines" multiple="1" display="no" altdistance="0.01" altunitdist="inch" altunit="inch"/>
+<grid distance="0.1" unitdist="inch" unit="inch" style="lines" multiple="1" display="no" altdistance="0.01" altunitdist="inch" altunit="inch"/>
 <layers>
 <layer number="1" name="Top" color="4" fill="1" visible="no" active="no"/>
@@
 <part name="U$5" library="vreg" deviceset="AP7361C-33E-13" device=""/>
 <part name="C5" library="rcl" deviceset="C-EU" device="C0805" value="4.7uF"/>
+<part name="R14" library="rcl" deviceset="R-EU_" device="R0603" value="1K"/>
+<part name="GND15" library="supply1" deviceset="GND" device=""/>
 </parts>
 <sheets>
@@
 <text x="-22.86" y="81.28" size="1.778" layer="91">Boot mode</text>
 <text x="60.96" y="93.98" size="1.778" layer="91">Boot mode</text>
+<text x="78.74" y="-5.08" size="1.778" layer="91">stops motor run in bootloader</text>
 </plain>
 <instances>
@@
 <instance part="U$5" gate="G$1" x="147.32" y="132.08"/>
 <instance part="C5" gate="G$1" x="173.99" y="121.92" rot="R180"/>
+<instance part="R14" gate="G$1" x="96.52" y="-7.62" rot="R180"/>
+<instance part="GND15" gate="1" x="106.68" y="-7.62" rot="R90"/>
 </instances>
 <busses>
@@
 <junction x="167.64" y="106.68"/>
 </segment>
+<segment>
+<pinref part="GND15" gate="1" pin="GND"/>
+<pinref part="R14" gate="G$1" pin="1"/>
+<wire x1="104.14" y1="-7.62" x2="101.6" y2="-7.62" width="0.1524" layer="91"/>
+</segment>
 </net>
 <net name="MOTOR1A" class="0">
@@
 <segment>
 <pinref part="U$4" gate="G$1" pin="INA"/>
-<wire x1="86.36" y1="-12.7" x2="99.06" y2="-12.7" width="0.1524" layer="91"/>
+<wire x1="86.36" y1="-12.7" x2="88.9" y2="-12.7" width="0.1524" layer="91"/>
 <label x="88.9" y="-12.7" size="1.778" layer="95"/>
-</segment>
-<segment>
+<pinref part="R14" gate="G$1" pin="2"/>
+<wire x1="88.9" y1="-12.7" x2="99.06" y2="-12.7" width="0.1524" layer="91"/>
+<wire x1="91.44" y1="-7.62" x2="88.9" y2="-7.62" width="0.1524" layer="91"/>
+<wire x1="88.9" y1="-7.62" x2="88.9" y2="-12.7" width="0.1524" layer="91"/>
+<junction x="88.9" y="-12.7"/>
+</segment>
+<segment>
